File: hardware/picstick.kicad_sch (KiCad schematic)
At the start: 15 parts, among them J1 USB_A, J2 AVR-ISP, J3 ICSP, U1 CH340E, U2 ATtiny44V-10M, U3 MCP1801T-3302I{slash}OT, Y1 TBD

Commit message: Updated schematic with crystal and LED component values.
Other:
- note added: "*16MHz"
- note added: "*ATtiny44V doesn't officially support clock speeds over 8MHz"
- note added: "0-5Ω"
- note added: "0Ω"
- note added: "12pF"
- note added: "150060BS75000"
- note added: "28pF"
- note added: "60Ω"
- note added: "8MHz"
- note added: "B1911NG--20D000114U1930"
- note added: "B1931NB--20C006714U1930"
- note added: "Blue"
- note added: "C4, C5"
- note added: "Crystal Selection"
- note added: "D1"
- note added: "LED Selection"
- note added: "R1"
- note added: "RH100-16.000-8-2020-TR"
- note added: "RH100-8.000-16-3030-TR-NS1"
- note added: "Y1"
- note added: "Yellow/Green"
- moved on the sheet: J3
